Commit message: feat: contact sensors on robot's foot links
- Add four contact sensors on each robot's foot link
- Format files in urdf and worlds directories
- Add Gazebo tags in unitree_go2_gazebo.xacro so that Gazebo does not
lumps fixed foot links with lower legs

File: unitree_go2_description/urdf/leg.xacro (robot description, xacro)
@@ -1,28 +1,29 @@
 <?xml version="1.0"?>
 <robot xmlns:xacro="http://www.ros.org/wiki/xacro">
-    <!-- <xacro:include filename="$(find unitree_go2_description)/transmission.xacro"/> -->
     <xacro:macro name="leg" params="name mirror mirror_dae front_hind front_hind_dae">
         <joint name="${name}_hip_joint" type="revolute">
             <xacro:if value="${(mirror_dae == False) and (front_hind_dae == True)}">
-                <origin rpy="0 0 0" xyz="${leg_offset_x} ${-leg_offset_y} 0"/>
+                <origin rpy="0 0 0" xyz="${leg_offset_x} ${-leg_offset_y} 0" />
             </xacro:if>
             <xacro:if value="${(mirror_dae == True) and (front_hind_dae == True)}">
-                <origin rpy="0 0 0" xyz="${leg_offset_x} ${leg_offset_y} 0"/>
+                <origin rpy="0 0 0" xyz="${leg_offset_x} ${leg_offset_y} 0" />
             </xacro:if>
             <xacro:if value="${(mirror_dae == False) and (front_hind_dae == False)}">
-                <origin rpy="0 0 0" xyz="${-leg_offset_x} ${-leg_offset_y} 0"/>
+                <origin rpy="0 0 0" xyz="${-leg_offset_x} ${-leg_offset_y} 0" />
             </xacro:if>
             <xacro:if value="${(mirror_dae == True) and (front_hind_dae == False)}">
-                <origin rpy="0 0 0" xyz="${-leg_offset_x} ${leg_offset_y} 0"/>
+                <origin rpy="0 0 0" xyz="${-leg_offset_x} ${leg_offset_y} 0" />
             </xacro:if>
-            <parent link="trunk"/>
-            <child link="${name}_hip_link"/>
-            <axis xyz="1 0 0"/>
-            <dynamics damping="${damping}" friction="${friction}"/>
+            <parent link="trunk" />
+            <child link="${name}_hip_link" />
+            <axis xyz="1 0 0" />
+            <dynamics damping="${damping}" friction="${friction}" />
             <xacro:if value="${(mirror_dae == True)}">
-                <limit effort="${hip_torque_max}" velocity="${hip_velocity_max}" lower="${hip_position_min}" upper="${hip_position_max}"/>
+                <limit effort="${hip_torque_max}" velocity="${hip_velocity_max}"
+                    lower="${hip_position_min}" upper="${hip_position_max}" />
             </xacro:if>
             <xacro:if value="${(mirror_dae == False)}">
-                <limit effort="${hip_torque_max}" velocity="${hip_velocity_max}" lower="${-hip_position_max}" upper="${-hip_position_min}"/>
+                <limit effort="${hip_torque_max}" velocity="${hip_velocity_max}"
+                    lower="${-hip_position_max}" upper="${-hip_position_min}" />
             </xacro:if>
         </joint>
@@ -30,127 +31,130 @@
             <visual>
                 <xacro:if value="${(mirror_dae == True) and (front_hind_dae == True)}">
-                    <origin rpy="0 0 0" xyz="0 0 0"/>
+                    <origin rpy="0 0 0" xyz="0 0 0" />
                 </xacro:if>
                 <xacro:if value="${(mirror_dae == False) and (front_hind_dae == True)}">
-                    <origin rpy="${PI} 0 0" xyz="0 0 0"/>
+                    <origin rpy="${PI} 0 0" xyz="0 0 0" />
                 </xacro:if>
                 <xacro:if value="${(mirror_dae == True) and (front_hind_dae == False)}">
-                    <origin rpy="0 ${PI} 0" xyz="0 0 0"/>
+                    <origin rpy="0 ${PI} 0" xyz="0 0 0" />
                 </xacro:if>
                 <xacro:if value="${(mirror_dae == False) and (front_hind_dae == False)}">
-                    <origin rpy="${PI} ${PI} 0" xyz="0 0 0"/>
+                    <origin rpy="${PI} ${PI} 0" xyz="0 0 0" />
                 </xacro:if>
                 <geometry>
-                    <mesh filename="file://$(find unitree_go2_description)/meshes/hip.dae" scale="1 1 1"/>
+                    <mesh filename="file://$(find unitree_go2_description)/meshes/hip.dae"
+                        scale="1 1 1" />
                 </geometry>
-                <!-- <material name="orange"/> -->
             </visual>
             <collision>
-                <origin rpy="${PI/2.0} 0 0" xyz="0 ${hip_offset*mirror} 0"/>
+                <origin rpy="${PI/2.0} 0 0" xyz="0 ${hip_offset*mirror} 0" />
                 <geometry>
-                    <cylinder length="${hip_length}" radius="${hip_radius}"/>
+                    <cylinder length="${hip_length}" radius="${hip_radius}" />
                 </geometry>
             </collision>
             <inertial>
-                <origin rpy="0 0 0" xyz="${hip_com_x*front_hind} ${hip_com_y*mirror} ${hip_com_z}"/>
-                <mass value="${hip_mass}"/>
+                <origin rpy="0 0 0" xyz="${hip_com_x*front_hind} ${hip_com_y*mirror} ${hip_com_z}" />
+                <mass value="${hip_mass}" />
                 <inertia
                     ixx="${hip_ixx}" ixy="${hip_ixy*mirror*front_hind}" ixz="${hip_ixz*front_hind}"
                     iyy="${hip_iyy}" iyz="${hip_iyz*mirror}"
-                    izz="${hip_izz}"/>
+                    izz="${hip_izz}" />
             </inertial>
         </link>
         <joint name="${name}_upper_leg_joint" type="revolute">
-            <origin rpy="0 0 0" xyz="0 ${thigh_offset*mirror} 0"/>
-            <parent link="${name}_hip_link"/>
-            <child link="${name}_upper_leg_link"/>
-            <axis xyz="0 1 0"/>
-            <dynamics damping="${damping}" friction="${friction}"/>
-            <limit effort="${thigh_torque_max}" velocity="${thigh_velocity_max}" lower="${thigh_position_min}" upper="${thigh_position_max}"/>
+            <origin rpy="0 0 0" xyz="0 ${thigh_offset*mirror} 0" />
+            <parent link="${name}_hip_link" />
+            <child link="${name}_upper_leg_link" />
+            <axis xyz="0 1 0" />
+            <dynamics damping="${damping}" friction="${friction}" />
+            <limit effort="${thigh_torque_max}" velocity="${thigh_velocity_max}"
+                lower="${thigh_position_min}" upper="${thigh_position_max}" />
         </joint>
         <link name="${name}_upper_leg_link">
             <visual>
-                <origin rpy="0 0 0" xyz="0 0 0"/>
+                <origin rpy="0 0 0" xyz="0 0 0" />
                 <geometry>
                     <xacro:if value="${mirror_dae == True}">
-                        <mesh filename="file://$(find unitree_go2_description)/meshes/thigh.dae" scale="1 1 1"/>
+                        <mesh filename="file://$(find unitree_go2_description)/meshes/thigh.dae"
+                            scale="1 1 1" />
                     </xacro:if>
                     <xacro:if value="${mirror_dae == False}">
-                        <mesh filename="file://$(find unitree_go2_description)/meshes/thigh_mirror.dae" scale="1 1 1"/>
+                        <mesh
+                            filename="file://$(find unitree_go2_description)/meshes/thigh_mirror.dae"
+                            scale="1 1 1" />
                     </xacro:if>
                 </geometry>
-                <!-- <material name="orange"/> -->
             </visual>
             <collision>
-                <origin rpy="0 ${PI/2.0} 0" xyz="0 0 ${-thigh_length/2.0}"/>
+                <origin rpy="0 ${PI/2.0} 0" xyz="0 0 ${-thigh_length/2.0}" />
                 <geometry>
-                    <box size="${thigh_length} ${thigh_width} ${thigh_height}"/>
+                    <box size="${thigh_length} ${thigh_width} ${thigh_height}" />
                 </geometry>
             </collision>
             <inertial>
-                <origin rpy="0 0 0" xyz="${thigh_com_x} ${thigh_com_y*mirror} ${thigh_com_z}"/>
-                <mass value="${thigh_mass}"/>
+                <origin rpy="0 0 0" xyz="${thigh_com_x} ${thigh_com_y*mirror} ${thigh_com_z}" />
+                <mass value="${thigh_mass}" />
                 <inertia
                     ixx="${thigh_ixx}" ixy="${thigh_ixy*mirror}" ixz="${thigh_ixz}"
                     iyy="${thigh_iyy}" iyz="${thigh_iyz*mirror}"
-                    izz="${thigh_izz}"/>
+                    izz="${thigh_izz}" />
             </inertial>
         </link>
         <joint name="${name}_lower_leg_joint" type="revolute">
-            <origin rpy="0 0 0" xyz="0 0 ${-thigh_length}"/>
-            <parent link="${name}_upper_leg_link"/>
-            <child link="${name}_lower_leg_link"/>
-            <axis xyz="0 1 0"/>
-            <dynamics damping="${damping}" friction="${friction}"/>
-            <limit effort="${calf_torque_max}" velocity="${calf_velocity_max}" lower="${calf_position_min}" upper="${calf_position_max}"/>
+            <origin rpy="0 0 0" xyz="0 0 ${-thigh_length}" />
+            <parent link="${name}_upper_leg_link" />
+            <child link="${name}_lower_leg_link" />
+            <axis xyz="0 1 0" />
+            <dynamics damping="${damping}" friction="${friction}" />
+            <limit effort="${calf_torque_max}" velocity="${calf_velocity_max}"
+                lower="${calf_position_min}" upper="${calf_position_max}" />
         </joint>
         <link name="${name}_lower_leg_link">
             <visual>
-                <origin rpy="0 0 0" xyz="0 0 0"/>
+                <origin rpy="0 0 0" xyz="0 0 0" />
                 <geometry>
-                    <mesh filename="file://$(find unitree_go2_description)/meshes/calf.dae" scale="1 1 1"/>
+                    <mesh filename="file://$(find unitree_go2_description)/meshes/calf.dae"
+                        scale="1 1 1" />
                 </geometry>
-                <!-- <material name="orange"/> -->
             </visual>
             <collision>
-                <origin rpy="0 ${PI/2.0} 0" xyz="0 0 ${-calf_length/2.0}"/>
+                <origin rpy="0 ${PI/2.0} 0" xyz="0 0 ${-calf_length/2.0}" />
                 <geometry>
-                    <box size="${calf_length} ${calf_width} ${calf_height}"/>
+                    <box size="${calf_length} ${calf_width} ${calf_height}" />
                 </geometry>
             </collision>
             <inertial>
-                <origin rpy="0 0 0" xyz="${calf_com_x} ${calf_com_y} ${calf_com_z}"/>
-                <mass value="${calf_mass}"/>
+                <origin rpy="0 0 0" xyz="${calf_com_x} ${calf_com_y} ${calf_com_z}" />
+                <mass value="${calf_mass}" />
                 <inertia
                     ixx="${calf_ixx}" ixy="${calf_ixy}" ixz="${calf_ixz}"
                     iyy="${calf_iyy}" iyz="${calf_iyz}"
-                    izz="${calf_izz}"/>
+                    izz="${calf_izz}" />
             </inertial>
         </link>
-        <joint name="${name}_foot_joint" type="fixed">0
-            <origin rpy="0 0 0" xyz="0 0 ${-(calf_length)}"/>
-            <parent link="${name}_lower_leg_link"/>
-            <child link="${name}_foot_link"/>
+        <joint name="${name}_foot_joint" type="fixed">
+            <origin rpy="0 0 0" xyz="0 0 ${-(calf_length)}" />
+            <parent link="${name}_lower_leg_link" />
+            <child link="${name}_foot_link" />
         </joint>
         <link name="${name}_foot_link">
             <visual>
-                <origin rpy="0 0 0" xyz="0 0 0"/>
+                <origin rpy="0 0 0" xyz="0 0 0" />
                 <geometry>
-                    <sphere radius="${foot_radius-0.01}"/>
+                    <sphere radius="${foot_radius-0.01}" />
                 </geometry>
-                <!-- <material name="orange"/> -->
             </visual>
             <collision>
-                <origin rpy="0 0 0" xyz="0 0 0"/>
+                <origin rpy="0 0 0" xyz="0 0 0" />
                 <geometry>
-                    <sphere radius="${foot_radius}"/>
+                    <sphere radius="${foot_radius}" />
                 </geometry>
             </collision>
             <inertial>
-                <mass value="${foot_mass}"/>
+                <mass value="${foot_mass}" />
                 <inertia
                     ixx="${(2*foot_mass)/5.0*(foot_radius*foot_radius)}" ixy="0.0" ixz="0.0"
                     iyy="${(2*foot_mass)/5.0*(foot_radius*foot_radius)}" iyz="0.0"
-                    izz="${(2*foot_mass)/5.0*(foot_radius*foot_radius)}"/>
+                    izz="${(2*foot_mass)/5.0*(foot_radius*foot_radius)}" />
             </inertial>
         </link>
@@ -160,20 +164,19 @@
             </hardware>
             <joint name="${name}_hip_joint">
-                <command_interface name="effort"/>
-                <state_interface name="position"/>
-                <state_interface name="velocity"/>
+                <command_interface name="effort" />
+                <state_interface name="position" />
+                <state_interface name="velocity" />
             </joint>
             <joint name="${name}_upper_leg_joint">
-                <command_interface name="effort"/>
-                <state_interface name="position"/>
-                <state_interface name="velocity"/>
+                <command_interface name="effort" />
+                <state_interface name="position" />
+                <state_interface name="velocity" />
             </joint>
             <joint name="${name}_lower_leg_joint">
-                <command_interface name="effort"/>
-                <state_interface name="position"/>
-                <state_interface name="velocity"/>
+                <command_interface name="effort" />
+                <state_interface name="position" />
+                <state_interface name="velocity" />
             </joint>
         </ros2_control>
-        <!-- <xacro:leg_transmission name="${name}"/> -->
     </xacro:macro>
 </robot>

File: unitree_go2_description/urdf/lidar_4D_lidar.xacro (robot description, xacro)
@@ -4,32 +4,34 @@
     <link name="lidar_l1_link">
         <inertial>
-            <mass value="0.5"/>
-            <origin rpy="0 0 0" xyz="0 0 0"/>
-            <inertia ixx="0.01" ixy="0" ixz="0" iyy="0.01" iyz="0" izz="0.01"/>
+            <mass value="0.5" />
+            <origin rpy="0 0 0" xyz="0 0 0" />
+            <inertia ixx="0.01" ixy="0" ixz="0" iyy="0.01" iyz="0" izz="0.01" />
         </inertial>
         <visual>
-            <origin rpy="0 0 0" xyz="0 0 0"/>
+            <origin rpy="0 0 0" xyz="0 0 0" />
             <geometry>
-                <mesh filename="file://$(find unitree_go2_description)/meshes/L1_4D_Lidar.dae" scale="1 1 1"/>
+                <mesh filename="file://$(find unitree_go2_description)/meshes/L1_4D_Lidar.dae"
+                    scale="1 1 1" />
             </geometry>
             <material name="black">
-                <color rgba="0.0 0.0 0.0 1.0"/>
+                <color rgba="0.0 0.0 0.0 1.0" />
             </material>
         </visual>
         <collision>
-            <origin rpy="0 0 0" xyz="0 0 0"/>
+            <origin rpy="0 0 0" xyz="0 0 0" />
             <geometry>
-                <mesh filename="file://$(find unitree_go2_description)/meshes/L1_4D_Lidar.dae" scale="1 1 1"/>
+                <mesh filename="file://$(find unitree_go2_description)/meshes/L1_4D_Lidar.dae"
+                    scale="1 1 1" />
             </geometry>
             <material name="black">
-                <color rgba="0.0 0.0 0.0 1.0"/>
+                <color rgba="0.0 0.0 0.0 1.0" />
             </material>
         </collision>
     </link>
     <joint name="lidar_l1_joint" type="fixed">
-        <parent link="base_link"/>
-        <child link="lidar_l1_link"/>
+        <parent link="base_link" />
+        <child link="lidar_l1_link" />
         <!-- <origin rpy="2.94 0 1.5705" xyz="0.25 -0.038 -0.03"/> -->
-        <origin rpy="2.879 0.0 1.5705" xyz="0.25 -0.038 -0.03"/>
+        <origin rpy="2.879 0.0 1.5705" xyz="0.25 -0.038 -0.03" />
     </joint>
     <gazebo reference="lidar_l1_link">

File: unitree_go2_description/urdf/materials.xacro (robot description, xacro)
@@ -2,29 +2,29 @@
 <robot>
     <material name="black">
-        <color rgba="0.0 0.0 0.0 1.0"/>
+        <color rgba="0.0 0.0 0.0 1.0" />
     </material>
     <material name="blue">
-        <color rgba="0.0 0.0 0.8 1.0"/>
+        <color rgba="0.0 0.0 0.8 1.0" />
     </material>
     <material name="green">
-        <color rgba="0.0 0.8 0.0 1.0"/>
+        <color rgba="0.0 0.8 0.0 1.0" />
     </material>
     <material name="grey">
-        <color rgba="0.2 0.2 0.2 0.0"/>
+        <color rgba="0.2 0.2 0.2 0.0" />
     </material>
     <material name="silver">
-        <color rgba="${233/255} ${233/255} ${216/255} 1.0"/>
+        <color rgba="${233/255} ${233/255} ${216/255} 1.0" />
     </material>
     <material name="orange">
-        <color rgba="${255/255} ${108/255} ${10/255} 1.0"/>
+        <color rgba="${255/255} ${108/255} ${10/255} 1.0" />
     </material>
     <material name="brown">
-        <color rgba="${222/255} ${207/255} ${195/255} 1.0"/>
+        <color rgba="${222/255} ${207/255} ${195/255} 1.0" />
     </material>
     <material name="red">
-        <color rgba="0.8 0.0 0.0 1.0"/>
+        <color rgba="0.8 0.0 0.0 1.0" />
     </material>
     <material name="white">
-        <color rgba="1.0 1.0 1.0 1.0"/>
+        <color rgba="1.0 1.0 1.0 1.0" />
     </material>
 </robot>

File: unitree_go2_description/urdf/unitree_go2_gazebo.xacro (robot description, xacro)
@@ -145,7 +145,17 @@
             <mu1>0.6</mu1>
             <mu2>0.6</mu2>
-            <self_collide>1</self_collide>
-            <kp>10000.0</kp>
-            <kd>1.0</kd>
+            <kp>10000.0</kp>
+            <kd>1.0</kd>
+            <sensor name="lf_foot_contact_sensor" type="contact">
+                <always_on>true</always_on>
+                <update_rate>100.0</update_rate>
+                <contact>
+                    <collision>lf_foot_link_collision</collision>
+                    <topic>/lf_foot_contacts</topic>
+                </contact>
+            </sensor>
+        </gazebo>
+        <gazebo reference="lf_foot_joint">
+            <preserveFixedJoint>true</preserveFixedJoint>
         </gazebo>
         <!-- FR leg -->
@@ -169,7 +179,17 @@
             <mu1>0.6</mu1>
             <mu2>0.6</mu2>
-            <self_collide>1</self_collide>
-            <kp>10000.0</kp>
-            <kd>1.0</kd>
+            <kp>10000.0</kp>
+            <kd>1.0</kd>
+            <sensor name="rf_foot_contact_sensor" type="contact">
+                <always_on>true</always_on>
+                <update_rate>100.0</update_rate>
+                <contact>
+                    <collision>rf_foot_link_collision</collision>
+                    <topic>/rf_foot_contacts</topic>
+                </contact>
+            </sensor>
+        </gazebo>
+        <gazebo reference="rf_foot_joint">
+            <preserveFixedJoint>true</preserveFixedJoint>
         </gazebo>
         <!-- RL leg -->
@@ -193,7 +213,17 @@
             <mu1>0.6</mu1>
             <mu2>0.6</mu2>
-            <self_collide>1</self_collide>
-            <kp>10000.0</kp>
-            <kd>1.0</kd>
+            <kp>10000.0</kp>
+            <kd>1.0</kd>
+            <sensor name="lh_foot_contact_sensor" type="contact">
+                <always_on>true</always_on>
+                <update_rate>100.0</update_rate>
+                <contact>
+                    <collision>lh_foot_link_collision</collision>
+                    <topic>/lh_foot_contacts</topic>
+                </contact>
+            </sensor>
+        </gazebo>
+        <gazebo reference="lh_foot_joint">
+            <preserveFixedJoint>true</preserveFixedJoint>
         </gazebo>
         <!-- RR leg -->
@@ -217,7 +247,17 @@
             <mu1>0.6</mu1>
             <mu2>0.6</mu2>
-            <self_collide>1</self_collide>
-            <kp>10000.0</kp>
-            <kd>1.0</kd>
+            <kp>10000.0</kp>
+            <kd>1.0</kd>
+            <sensor name="rh_foot_contact_sensor" type="contact">
+                <always_on>true</always_on>
+                <update_rate>100.0</update_rate>
+                <contact>
+                    <collision>rh_foot_link_collision</collision>
+                    <topic>/rh_foot_contacts</topic>
+                </contact>
+            </sensor>
+        </gazebo>
+        <gazebo reference="rh_foot_joint">
+            <preserveFixedJoint>true</preserveFixedJoint>
         </gazebo>
     </xacro:macro>
