Commit message: feat: contact sensors on robot's foot links
- Add four contact sensors on each robot's foot link
- Format files in urdf and worlds directories
- Add Gazebo tags in unitree_go2_gazebo.xacro so that Gazebo does not
lumps fixed foot links with lower legs

File: unitree_go2_description/urdf/velodyne.xacro (robot description, xacro)
@@ -2,46 +2,47 @@
 <robot xmlns:xacro="http://www.ros.org/wiki/xacro">
     <joint name="velodyne_base_mount_joint" type="fixed">
-        <origin rpy="0 0 0" xyz="0.2 0 0.08"/>
-        <parent link="base_link"/>
-        <child link="velodyne_base_link"/>
+        <origin rpy="0 0 0" xyz="0.2 0 0.08" />
+        <parent link="base_link" />
+        <child link="velodyne_base_link" />
     </joint>
     <link name="velodyne_base_link">
         <inertial>
-            <mass value="0.83"/>
-            <origin xyz="0 0 0.03585"/>
-            <inertia ixx="0.000908059425" ixy="0" ixz="0" iyy="0.000908059425" iyz="0" izz="0.0011049624"/>
+            <mass value="0.83" />
+            <origin xyz="0 0 0.03585" />
+            <inertia ixx="0.000908059425" ixy="0" ixz="0" iyy="0.000908059425" iyz="0"
+                izz="0.0011049624" />
         </inertial>
         <visual>
             <geometry>
-                <mesh filename="file://$(find unitree_go2_description)/meshes/VLP16_base_1.dae"/>
+                <mesh filename="file://$(find unitree_go2_description)/meshes/VLP16_base_1.dae" />
             </geometry>
         </visual>
         <visual>
             <geometry>
-                <mesh filename="file://$(find unitree_go2_description)/meshes/VLP16_base_2.dae"/>
+                <mesh filename="file://$(find unitree_go2_description)/meshes/VLP16_base_2.dae" />
             </geometry>
         </visual>
         <collision>
-            <origin rpy="0 0 0" xyz="0 0 0.03585"/>
+            <origin rpy="0 0 0" xyz="0 0 0.03585" />
             <geometry>
-                <cylinder length="0.0717" radius="0.0516"/>
+                <cylinder length="0.0717" radius="0.0516" />
             </geometry>
         </collision>
     </link>
     <joint name="velodyne_base_scan_joint" type="fixed">
-        <origin rpy="0 0 0" xyz="0 0 0.0377"/>
-        <parent link="velodyne_base_link"/>
-        <child link="velodyne"/>
+        <origin rpy="0 0 0" xyz="0 0 0.0377" />
+        <parent link="velodyne_base_link" />
+        <child link="velodyne" />
     </joint>
     <link name="velodyne">
         <inertial>
-            <mass value="0.01"/>
-            <origin xyz="0 0 0"/>
-            <inertia ixx="1e-7" ixy="0" ixz="0" iyy="1e-7" iyz="0" izz="1e-7"/>
+            <mass value="0.01" />
+            <origin xyz="0 0 0" />
+            <inertia ixx="1e-7" ixy="0" ixz="0" iyy="1e-7" iyz="0" izz="1e-7" />
         </inertial>
         <visual>
-            <origin xyz="0 0 -0.0377"/>
+            <origin xyz="0 0 -0.0377" />
             <geometry>
-                <mesh filename="file://$(find unitree_go2_description)/meshes/VLP16_scan.dae"/>
+                <mesh filename="file://$(find unitree_go2_description)/meshes/VLP16_scan.dae" />
             </geometry>
         </visual>
