Commit message: feat(urdf): add argument to choose between effort or position command interfaces
Add command_interface argument in unitree_go2_robot.xacro to choose the
joints' command interface inside ros2_control tags. The argument can be
either effort or position. The default if effort, so the change is
backward compatible.

File: unitree_go2_description/urdf/leg.xacro (robot description, xacro)
@@ -1,5 +1,6 @@
 <?xml version="1.0"?>
 <robot xmlns:xacro="http://www.ros.org/wiki/xacro">
-    <xacro:macro name="leg" params="name mirror mirror_dae front_hind front_hind_dae">
+    <xacro:macro name="leg"
+        params="name mirror mirror_dae front_hind front_hind_dae command_interface:=effort">
         <joint name="${name}_hip_joint" type="revolute">
             <xacro:if value="${(mirror_dae == False) and (front_hind_dae == True)}">
@@ -163,19 +164,38 @@
                 <plugin>gz_ros2_control/GazeboSimSystem</plugin>
             </hardware>
-            <joint name="${name}_hip_joint">
-                <command_interface name="effort" />
-                <state_interface name="position" />
-                <state_interface name="velocity" />
-            </joint>
-            <joint name="${name}_upper_leg_joint">
-                <command_interface name="effort" />
-                <state_interface name="position" />
-                <state_interface name="velocity" />
-            </joint>
-            <joint name="${name}_lower_leg_joint">
-                <command_interface name="effort" />
-                <state_interface name="position" />
-                <state_interface name="velocity" />
-            </joint>
+            <xacro:if value="${command_interface == 'effort'}">
+                <joint name="${name}_hip_joint">
+                    <command_interface name="effort" />
+                    <state_interface name="position" />
+                    <state_interface name="velocity" />
+                </joint>
+                <joint name="${name}_upper_leg_joint">
+                    <command_interface name="effort" />
+                    <state_interface name="position" />
+                    <state_interface name="velocity" />
+                </joint>
+                <joint name="${name}_lower_leg_joint">
+                    <command_interface name="effort" />
+                    <state_interface name="position" />
+                    <state_interface name="velocity" />
+                </joint>
+            </xacro:if>
+            <xacro:if value="${command_interface == 'position'}">
+                <joint name="${name}_hip_joint">
+                    <command_interface name="position" />
+                    <state_interface name="position" />
+                    <state_interface name="velocity" />
+                </joint>
+                <joint name="${name}_upper_leg_joint">
+                    <command_interface name="position" />
+                    <state_interface name="position" />
+                    <state_interface name="velocity" />
+                </joint>
+                <joint name="${name}_lower_leg_joint">
+                    <command_interface name="position" />
+                    <state_interface name="position" />
+                    <state_interface name="velocity" />
+                </joint>
+            </xacro:if>
         </ros2_control>
     </xacro:macro>

File: unitree_go2_description/urdf/unitree_go2_robot.xacro (robot description, xacro)
@@ -1,6 +1,6 @@
 <?xml version="1.0"?>
-<robot name="go2"
-    xmlns:xacro="http://www.ros.org/wiki/xacro">
+<robot name="go2" xmlns:xacro="http://www.ros.org/wiki/xacro">
     <xacro:arg name="DEBUG" default="false" />
+    <xacro:arg name="command_interface" default="effort" />
     <xacro:arg name="robot_controllers"
         default="$(find unitree_go2_sim)/config/ros_control/ros_control.yaml" />
@@ -8,14 +8,8 @@
     <xacro:include filename="$(find unitree_go2_description)/urdf/materials.xacro" />
     <xacro:include filename="$(find unitree_go2_description)/urdf/leg.xacro" />
-    <!-- <xacro:include filename="$(find unitree_go2_description)/stairs.xacro"/> -->
     <xacro:include filename="$(find unitree_go2_description)/urdf/unitree_go2_gazebo.xacro" />
-    <!-- <xacro:include filename="$(find unitree_go2_description)/launch/stairs.urdf.xacro"/> -->
     <xacro:include filename="$(find unitree_go2_description)/urdf/velodyne.xacro" />
     <xacro:include filename="$(find unitree_go2_description)/urdf/lidar_4D_lidar.xacro" />
-    <!-- <xacro:stairs stairs="15" xpos="0" ypos="0" zpos="0" /> -->
     <xacro:unitree_go2_gazebo robot_controllers="$(arg robot_controllers)" />
-    <!-- Rotor related joint and link is only for demonstrate location. -->
-    <!-- Actually, the rotor will rotate and the joint is not fixed. Reduction ratio should be
-    considered. -->
     <!-- Debug mode will hung up the robot, use "true" or "false" to switch it. -->
     <xacro:if value="$(arg DEBUG)">
@@ -113,37 +107,11 @@
         <origin rpy="0 0 0" xyz="0.326 0 0.043" />
     </joint>
-    <!-- <joint name="lidar_l1_joint" type="fixed">
-        <parent link="base_link"/>
-        <child link="lidar_l1_link"/>
-        <origin rpy="2.94 0 1.5705" xyz="0.25 -0.038 -0.03"/>
-    </joint>
-    <link name="lidar_l1_link">
-        <inertial>
-            <mass value="0.5"/>
-            <origin rpy="0 0 0" xyz="0 0 0"/>
-            <inertia ixx="0.01" ixy="0" ixz="0" iyy="0.01" iyz="0" izz="0.01"/>
-        </inertial>
-        <visual>
-            <origin rpy="0 0 0" xyz="0 0 0"/>
-            <geometry>
-                <mesh filename="file://$(find unitree_go2_description)/meshes/L1_4D_Lidar.dae" scale="1 1 1"/>
-            </geometry>
-            <material name="black">
-                <color rgba="0.0 0.0 0.0 1.0"/>
-            </material>
-        </visual>
-        <collision>
-            <origin rpy="0 0 0" xyz="0 0 0"/>
-            <geometry>
-                <mesh filename="file://$(find unitree_go2_description)/meshes/L1_4D_Lidar.dae" scale="1 1 1"/>
-            </geometry>
-            <material name="black">
-                <color rgba="0.0 0.0 0.0 1.0"/>
-            </material>
-        </collision>
-    </link> -->
-    <xacro:leg name="rf" mirror="-1" mirror_dae="False" front_hind="1" front_hind_dae="True" />
-    <xacro:leg name="lf" mirror="1" mirror_dae="True" front_hind="1" front_hind_dae="True" />
-    <xacro:leg name="rh" mirror="-1" mirror_dae="False" front_hind="-1" front_hind_dae="False" />
-    <xacro:leg name="lh" mirror="1" mirror_dae="True" front_hind="-1" front_hind_dae="False" />
+    <xacro:leg name="rf" mirror="-1" mirror_dae="False" front_hind="1" front_hind_dae="True"
+        command_interface="$(arg command_interface)" />
+    <xacro:leg name="lf" mirror="1" mirror_dae="True" front_hind="1" front_hind_dae="True"
+        command_interface="$(arg command_interface)" />
+    <xacro:leg name="rh" mirror="-1" mirror_dae="False" front_hind="-1" front_hind_dae="False"
+        command_interface="$(arg command_interface)" />
+    <xacro:leg name="lh" mirror="1" mirror_dae="True" front_hind="-1" front_hind_dae="False"
+        command_interface="$(arg command_interface)" />
 </robot>
