Commit message: feat(urdf): add arguments to disable camera, lidar L1 and velodyne lidar
Arguments are false by default, so the feature is backward compatible

File: unitree_go2_description/urdf/lidar_4D_lidar.xacro (robot description, xacro)
@@ -1,72 +1,72 @@
 <?xml version="1.0"?>
 <robot xmlns:xacro="http://www.ros.org/wiki/xacro">
-    <!-- Lidar L1-->
-    <link name="lidar_l1_link">
-        <inertial>
-            <mass value="0.5" />
-            <origin rpy="0 0 0" xyz="0 0 0" />
-            <inertia ixx="0.01" ixy="0" ixz="0" iyy="0.01" iyz="0" izz="0.01" />
-        </inertial>
-        <visual>
-            <origin rpy="0 0 0" xyz="0 0 0" />
-            <geometry>
-                <mesh filename="file://$(find unitree_go2_description)/meshes/L1_4D_Lidar.dae"
-                    scale="1 1 1" />
-            </geometry>
-            <material name="black">
-                <color rgba="0.0 0.0 0.0 1.0" />
-            </material>
-        </visual>
-        <collision>
-            <origin rpy="0 0 0" xyz="0 0 0" />
-            <geometry>
-                <mesh filename="file://$(find unitree_go2_description)/meshes/L1_4D_Lidar.dae"
-                    scale="1 1 1" />
-            </geometry>
-            <material name="black">
-                <color rgba="0.0 0.0 0.0 1.0" />
-            </material>
-        </collision>
-    </link>
-    <joint name="lidar_l1_joint" type="fixed">
-        <parent link="base_link" />
-        <child link="lidar_l1_link" />
-        <!-- <origin rpy="2.94 0 1.5705" xyz="0.25 -0.038 -0.03"/> -->
-        <origin rpy="2.879 0.0 1.5705" xyz="0.25 -0.038 -0.03" />
-    </joint>
-    <gazebo reference="lidar_l1_link">
-        <sensor name="lidar_l1" type="gpu_lidar">
-            <topic>unitree_lidar</topic>
-            <update_rate>10</update_rate>
-            <lidar>
-                <scan>
-                    <horizontal>
-                        <samples>600</samples>
-                        <resolution>1</resolution>
-                        <min_angle>-3.14159</min_angle>
-                        <max_angle>3.14159</max_angle>
-                    </horizontal>
-                    <vertical>
-                        <samples>30</samples>
-                        <resolution>1</resolution>
-                        <min_angle>-0.785398</min_angle>
-                        <max_angle>0.785398</max_angle>
-                    </vertical>
-                </scan>
-                <range>
-                    <min>0.8</min>
-                    <max>30.0</max>
-                    <resolution>0.001</resolution>
-                </range>
-                <noise>
-                    <type>gaussian</type>
-                    <mean>0.0</mean>
-                    <stddev>0.008</stddev>
-                </noise>
-            </lidar>
-            <visualize>false</visualize>
-            <gz_frame_id>lidar_l1_link</gz_frame_id>
-            <always_on>1</always_on>
-        </sensor>
-    </gazebo>
+    <xacro:macro name="lidar_l1">
+        <link name="lidar_l1_link">
+            <inertial>
+                <mass value="0.5" />
+                <origin rpy="0 0 0" xyz="0 0 0" />
+                <inertia ixx="0.01" ixy="0" ixz="0" iyy="0.01" iyz="0" izz="0.01" />
+            </inertial>
+            <visual>
+                <origin rpy="0 0 0" xyz="0 0 0" />
+                <geometry>
+                    <mesh filename="file://$(find unitree_go2_description)/meshes/L1_4D_Lidar.dae"
+                        scale="1 1 1" />
+                </geometry>
+                <material name="black">
+                    <color rgba="0.0 0.0 0.0 1.0" />
+                </material>
+            </visual>
+            <collision>
+                <origin rpy="0 0 0" xyz="0 0 0" />
+                <geometry>
+                    <mesh filename="file://$(find unitree_go2_description)/meshes/L1_4D_Lidar.dae"
+                        scale="1 1 1" />
+                </geometry>
+                <material name="black">
+                    <color rgba="0.0 0.0 0.0 1.0" />
+                </material>
+            </collision>
+        </link>
+        <joint name="lidar_l1_joint" type="fixed">
+            <parent link="base_link" />
+            <child link="lidar_l1_link" />
+            <origin rpy="2.879 0.0 1.5705" xyz="0.25 -0.038 -0.03" />
+        </joint>
+        <gazebo reference="lidar_l1_link">
+            <sensor name="lidar_l1" type="gpu_lidar">
+                <topic>unitree_lidar</topic>
+                <update_rate>10</update_rate>
+                <lidar>
+                    <scan>
+                        <horizontal>
+                            <samples>600</samples>
+                            <resolution>1</resolution>
+                            <min_angle>-3.14159</min_angle>
+                            <max_angle>3.14159</max_angle>
+                        </horizontal>
+                        <vertical>
+                            <samples>30</samples>
+                            <resolution>1</resolution>
+                            <min_angle>-0.785398</min_angle>
+                            <max_angle>0.785398</max_angle>
+                        </vertical>
+                    </scan>
+                    <range>
+                        <min>0.8</min>
+                        <max>30.0</max>
+                        <resolution>0.001</resolution>
+                    </range>
+                    <noise>
+                        <type>gaussian</type>
+                        <mean>0.0</mean>
+                        <stddev>0.008</stddev>
+                    </noise>
+                </lidar>
+                <visualize>false</visualize>
+                <gz_frame_id>lidar_l1_link</gz_frame_id>
+                <always_on>1</always_on>
+            </sensor>
+        </gazebo>
+    </xacro:macro>
 </robot>

File: unitree_go2_description/urdf/unitree_go2_robot.xacro (robot description, xacro)
@@ -5,4 +5,7 @@
     <xacro:arg name="robot_controllers"
         default="$(find unitree_go2_sim)/config/ros_control/ros_control.yaml" />
+    <xacro:arg name="disable_camera" default="false" />
+    <xacro:arg name="disable_lidar_l1" default="false" />
+    <xacro:arg name="disable_velodyne_lidar" default="false" />
     <xacro:include filename="$(find unitree_go2_description)/urdf/const.xacro" />
     <xacro:include filename="$(find unitree_go2_description)/urdf/materials.xacro" />
@@ -21,4 +24,5 @@
         </joint>
     </xacro:if>
+    <!-- Base Link -->
     <link name="base_link">
         <visual>
@@ -29,9 +33,5 @@
         </visual>
     </link>
-    <joint name="floating_base" type="fixed">
-        <origin rpy="0 0 0" xyz="0 0 0" />
-        <parent link="base_link" />
-        <child link="trunk" />
-    </joint>
+    <!-- Trunk -->
     <link name="trunk">
         <visual>
@@ -55,9 +55,10 @@
         </inertial>
     </link>
-    <joint name="imu_joint" type="fixed">
-        <parent link="trunk" />
-        <child link="imu_link" />
+    <joint name="floating_base" type="fixed">
         <origin rpy="0 0 0" xyz="0 0 0" />
+        <parent link="base_link" />
+        <child link="trunk" />
     </joint>
+    <!-- IMU -->
     <link name="imu_link">
         <inertial>
@@ -79,32 +80,10 @@
         </collision>
     </link>
-    <!-- Camera Link-->
-    <link name="camera_link">
-        <inertial>
-            <mass value="0.001" />
-            <origin rpy="0 0 0" xyz="0 0 0" />
-            <inertia ixx="0.0001" ixy="0" ixz="0" iyy="0.0001" iyz="0" izz="0.0001" />
-        </inertial>
-        <visual>
-            <origin rpy="0 0 0" xyz="0 0 0" />
-            <geometry>
-                <sphere radius="0.001" />
-            </geometry>
-            <material name="">
-                <color rgba="0.5 0 0 1" />
-            </material>
-        </visual>
-        <collision>
-            <origin rpy="0 0 0" xyz="0 0 0" />
-            <geometry>
-                <sphere radius="0.001" />
-            </geometry>
-        </collision>
-    </link>
-    <joint name="camera_joint" type="fixed">
+    <joint name="imu_joint" type="fixed">
         <parent link="trunk" />
-        <child link="camera_link" />
-        <origin rpy="0 0 0" xyz="0.326 0 0.043" />
+        <child link="imu_link" />
+        <origin rpy="0 0 0" xyz="0 0 0" />
     </joint>
+    <!-- Legs -->
     <xacro:leg name="rf" mirror="-1" mirror_dae="False" front_hind="1" front_hind_dae="True"
         command_interface="$(arg command_interface)" />
@@ -115,3 +94,40 @@
     <xacro:leg name="lh" mirror="1" mirror_dae="True" front_hind="-1" front_hind_dae="False"
         command_interface="$(arg command_interface)" />
+    <!-- Camera -->
+    <xacro:unless value="$(arg disable_camera)">
+        <link name="camera_link">
+            <inertial>
+                <mass value="0.001" />
+                <origin rpy="0 0 0" xyz="0 0 0" />
+                <inertia ixx="0.0001" ixy="0" ixz="0" iyy="0.0001" iyz="0" izz="0.0001" />
+            </inertial>
+            <visual>
+                <origin rpy="0 0 0" xyz="0 0 0" />
+                <geometry>
+                    <sphere radius="0.001" />
+                </geometry>
+                <material name="">
+                    <color rgba="0.5 0 0 1" />
+                </material>
+            </visual>
+            <collision>
+                <origin rpy="0 0 0" xyz="0 0 0" />
+                <geometry>
+                    <sphere radius="0.001" />
+                </geometry>
+            </collision>
+        </link>
+        <joint name="camera_joint" type="fixed">
+            <parent link="trunk" />
+            <child link="camera_link" />
+            <origin rpy="0 0 0" xyz="0.326 0 0.043" />
+        </joint>
+    </xacro:unless>
+    <!-- LiDARs -->
+    <xacro:unless value="$(arg disable_lidar_l1)">
+        <xacro:lidar_l1 />
+    </xacro:unless>
+    <xacro:unless value="$(arg disable_velodyne_lidar)">
+        <xacro:velodyne_lidar />
+    </xacro:unless>
 </robot>

File: unitree_go2_description/urdf/velodyne.xacro (robot description, xacro)
@@ -1,87 +1,89 @@
 <?xml version="1.0"?>
 <robot xmlns:xacro="http://www.ros.org/wiki/xacro">
-    <joint name="velodyne_base_mount_joint" type="fixed">
-        <origin rpy="0 0 0" xyz="0.2 0 0.08" />
-        <parent link="base_link" />
-        <child link="velodyne_base_link" />
-    </joint>
-    <link name="velodyne_base_link">
-        <inertial>
-            <mass value="0.83" />
-            <origin xyz="0 0 0.03585" />
-            <inertia ixx="0.000908059425" ixy="0" ixz="0" iyy="0.000908059425" iyz="0"
-                izz="0.0011049624" />
-        </inertial>
-        <visual>
-            <geometry>
-                <mesh filename="file://$(find unitree_go2_description)/meshes/VLP16_base_1.dae" />
-            </geometry>
-        </visual>
-        <visual>
-            <geometry>
-                <mesh filename="file://$(find unitree_go2_description)/meshes/VLP16_base_2.dae" />
-            </geometry>
-        </visual>
-        <collision>
-            <origin rpy="0 0 0" xyz="0 0 0.03585" />
-            <geometry>
-                <cylinder length="0.0717" radius="0.0516" />
-            </geometry>
-        </collision>
-    </link>
-    <joint name="velodyne_base_scan_joint" type="fixed">
-        <origin rpy="0 0 0" xyz="0 0 0.0377" />
-        <parent link="velodyne_base_link" />
-        <child link="velodyne" />
-    </joint>
-    <link name="velodyne">
-        <inertial>
-            <mass value="0.01" />
-            <origin xyz="0 0 0" />
-            <inertia ixx="1e-7" ixy="0" ixz="0" iyy="1e-7" iyz="0" izz="1e-7" />
-        </inertial>
-        <visual>
-            <origin xyz="0 0 -0.0377" />
-            <geometry>
-                <mesh filename="file://$(find unitree_go2_description)/meshes/VLP16_scan.dae" />
-            </geometry>
-        </visual>
-    </link>
-    <!-- Gazebo Sim Velodyne Sensor plugin -->
-    <gazebo reference="velodyne">
-        <sensor name="velodyne-VLP16" type="gpu_lidar">
-            <topic>velodyne_points</topic>
-            <update_rate>10</update_rate>
-            <gz_frame_id>velodyne</gz_frame_id>
-            <lidar>
-                <scan>
-                    <horizontal>
-                        <samples>440</samples>
-                        <resolution>1</resolution>
-                        <min_angle>-3.14159</min_angle>
-                        <max_angle>3.14159</max_angle>
-                    </horizontal>
-                    <vertical>
-                        <samples>16</samples>
-                        <resolution>1</resolution>
-                        <min_angle>-0.261799</min_angle>
-                        <max_angle>0.261799</max_angle>
-                    </vertical>
-                </scan>
-                <range>
-                    <min>0.5</min>
-                    <max>131.0</max>
-                    <resolution>0.001</resolution>
-                </range>
-                <noise>
-                    <type>gaussian</type>
-                    <mean>0.0</mean>
-                    <stddev>0.008</stddev>
-                </noise>
-                <frame_id>velodyne</frame_id>
-            </lidar>
-            <visualize>true</visualize>
-            <always_on>1</always_on>
-        </sensor>
-    </gazebo>
+    <xacro:macro name="velodyne_lidar">
+        <link name="velodyne_base_link">
+            <inertial>
+                <mass value="0.83" />
+                <origin xyz="0 0 0.03585" />
+                <inertia ixx="0.000908059425" ixy="0" ixz="0" iyy="0.000908059425" iyz="0"
+                    izz="0.0011049624" />
+            </inertial>
+            <visual>
+                <geometry>
+                    <mesh filename="file://$(find unitree_go2_description)/meshes/VLP16_base_1.dae" />
+                </geometry>
+            </visual>
+            <visual>
+                <geometry>
+                    <mesh filename="file://$(find unitree_go2_description)/meshes/VLP16_base_2.dae" />
+                </geometry>
+            </visual>
+            <collision>
+                <origin rpy="0 0 0" xyz="0 0 0.03585" />
+                <geometry>
+                    <cylinder length="0.0717" radius="0.0516" />
+                </geometry>
+            </collision>
+        </link>
+        <joint name="velodyne_base_mount_joint" type="fixed">
+            <origin rpy="0 0 0" xyz="0.2 0 0.08" />
+            <parent link="base_link" />
+            <child link="velodyne_base_link" />
+        </joint>
+        <link name="velodyne">
+            <inertial>
+                <mass value="0.01" />
+                <origin xyz="0 0 0" />
+                <inertia ixx="1e-7" ixy="0" ixz="0" iyy="1e-7" iyz="0" izz="1e-7" />
+            </inertial>
+            <visual>
+                <origin xyz="0 0 -0.0377" />
+                <geometry>
+                    <mesh filename="file://$(find unitree_go2_description)/meshes/VLP16_scan.dae" />
+                </geometry>
+            </visual>
+        </link>
+        <joint name="velodyne_base_scan_joint" type="fixed">
+            <origin rpy="0 0 0" xyz="0 0 0.0377" />
+            <parent link="velodyne_base_link" />
+            <child link="velodyne" />
+        </joint>
+        <!-- Gazebo Sim Velodyne Sensor plugin -->
+        <gazebo reference="velodyne">
+            <sensor name="velodyne-VLP16" type="gpu_lidar">
+                <topic>velodyne_points</topic>
+                <update_rate>10</update_rate>
+                <gz_frame_id>velodyne</gz_frame_id>
+                <lidar>
+                    <scan>
+                        <horizontal>
+                            <samples>440</samples>
+                            <resolution>1</resolution>
+                            <min_angle>-3.14159</min_angle>
+                            <max_angle>3.14159</max_angle>
+                        </horizontal>
+                        <vertical>
+                            <samples>16</samples>
+                            <resolution>1</resolution>
+                            <min_angle>-0.261799</min_angle>
+                            <max_angle>0.261799</max_angle>
+                        </vertical>
+                    </scan>
+                    <range>
+                        <min>0.5</min>
+                        <max>131.0</max>
+                        <resolution>0.001</resolution>
+                    </range>
+                    <noise>
+                        <type>gaussian</type>
+                        <mean>0.0</mean>
+                        <stddev>0.008</stddev>
+                    </noise>
+                    <frame_id>velodyne</frame_id>
+                </lidar>
+                <visualize>true</visualize>
+                <always_on>1</always_on>
+            </sensor>
+        </gazebo>
+    </xacro:macro>
 </robot>
